File: Hardware-v2/kicad/audio-dommain.kicad_sch (KiCad schematic)
At the start: 45 parts, among them U13 ADAU1452, U14 25AA1024-I_SM, Y3 ABM3B-12.288MHZ-10-1-U-T

Commit message: Correct the v2 EEPROM footprint and crystal load capacitors
Compared the ADAU1452 section with the EVAL-ADAU1452REVBZ user guide
(UG-1662) and the ADAU1452 datasheet.

- U14: 25AA1024-I/SM is a 208 mil SOIJ-8, but it was on a 150 mil SOIC
  footprint. Use Package_SO:SOIC-8_5.3x5.3mm_P1.27mm and fix the PNM.
- C141/C142 (Y3): 15 pF NP0 instead of 12 pF X7R.
- C139/C140 (Y2): 12 pF NP0 instead of 12 pF X7R.
- C6: add 1 uF on 1V2 near U13 pin 20, which the datasheet asks for.
- Widen the 1V2 trace from U13 pin 20 to 0.35 mm.

Co-Authored-By: Claude Opus 5.5 (1M context) <noreply@anthropic.com>
Parts:
- added C6: 1uF, Capacitor_SMD:C_0603_1608Metric, symbol Device:C
- C141, C142: value 12pF -> 15pF; PNM C0603C120K5RACTU -> CC0603JRNPO9BN150
- U14: value 25AA1024-I_SM -> 25AA1024-I/SM; footprint MIKILAB_25AA1024:SOIC127P600X175-8N -> Package_SO:SOIC-8_5.3x5.3mm_P1.27mm; PNM 25AA1024-I_SM -> 25AA1024-I/SM
Connections:
- net 1V2: now also C6.1
- net GND: now also C6.2
Changed lines of the file:
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@@
 	)
 	(junction
+		(at 250.19 19.05)
+		(diameter 0)
+		(color 0 0 0 0)
+	)
+	(junction
 		(at 219.71 26.67)
 		(diameter 0)
@@
 	)
 	(junction
+		(at 242.57 26.67)
+		(diameter 0)
+		(color 0 0 0 0)
+	)
+	(junction
 		(at 218.44 123.19)
 		(diameter 0)
@@
 	(wire
 		(pts
+			(xy 242.57 26.67) (xy 250.19 26.67)
+		)
+		(stroke
+			(width 0)
+			(type default)
+		)
+	)
+	(wire
+		(pts
 			(xy 227.33 125.73) (xy 228.6 125.73)
 		)
@@
 	)
 	(symbol
+		(lib_id "Device:C")
+		(at 250.19 22.86 0)
+		(unit 1)
+		(body_style 1)
+		(exclude_from_sim no)
+		(in_bom yes)
+		(on_board yes)
+		(in_pos_files yes)
+		(dnp no)
+		(fields_autoplaced yes)
+		(property "Reference" "C6"
+			(at 254 21.5899 0)
+			(show_name no)
+			(do_not_autoplace no)
+			(effects
+				(font
+					(size 1.27 1.27)
+				)
+				(justify left)
+			)
+		)
+		(property "Value" "1uF"
+			(at 254 24.1299 0)
+			(show_name no)
+			(do_not_autoplace no)
+			(effects
+				(font
+					(size 1.27 1.27)
+				)
+				(justify left)
+			)
+		)
+		(property "Footprint" "Capacitor_SMD:C_0603_1608Metric"
+			(at 251.1552 26.67 0)
+			(hide yes)
+			(show_name no)
+			(do_not_autoplace no)
+			(effects
+				(font
+					(size 1.27 1.27)
+				)
+			)
+		)
+		(property "Datasheet" ""
+			(at 250.19 22.86 0)
+			(hide yes)
+			(show_name no)
+			(do_not_autoplace no)
+			(effects
+				(font
+					(size 1.27 1.27)
+				)
+			)
+		)
+		(property "Description" "CAP CER 1uF 50V X7R 0603"
+			(at 250.19 22.86 0)
+			(hide yes)
+			(show_name no)
+			(do_not_autoplace no)
+			(effects
+				(font
+					(size 1.27 1.27)
+				)
+			)
+		)
+		(property "PNM" "CL10B105KB8NQNC"
+			(at 250.19 22.86 0)
+			(hide yes)
+			(show_name no)
+			(do_not_autoplace no)
+			(effects
+				(font
+					(size 1.27 1.27)
+				)
+			)
+		)
+		(property "DIGIKEY-PURCHASE-URL" ""
+			(at 250.19 22.86 0)
+			(hide yes)
+			(show_name no)
+			(do_not_autoplace no)
+			(effects
+				(font
+					(size 1.27 1.27)
+				)
+			)
+		)
+		(property "MFANUFACTURER" ""
+			(at 250.19 22.86 0)
+			(hide yes)
+			(show_name no)
+			(do_not_autoplace no)
+			(effects
+				(font
+					(size 1.27 1.27)
+				)
+			)
+		)
+		(property "MOUSER-PURCHASE-URL" ""
+			(at 250.19 22.86 0)
+			(hide yes)
+			(show_name no)
+			(do_not_autoplace no)
+			(effects
+				(font
+					(size 1.27 1.27)
+				)
+			)
+		)
+		(property "TEXAS_INSTRUMENTS-PURCHASE-URL" ""
+			(at 250.19 22.86 0)
+			(hide yes)
+			(show_name no)
+			(do_not_autoplace no)
+			(effects
+				(font
+					(size 1.27 1.27)
+				)
+			)
+		)
+		(property "KLC_S3.3" ""
+			(at 250.19 22.86 0)
+			(hide yes)
+			(show_name no)
+			(do_not_autoplace no)
+			(effects
+				(font
+					(size 1.27 1.27)
+				)
+			)
+		)
+		(property "KLC_S4.1" ""
+			(at 250.19 22.86 0)
+			(hide yes)
+			(show_name no)
+			(do_not_autoplace no)
+			(effects
+				(font
+					(size 1.27 1.27)
+				)
+			)
+		)
+		(property "SNAPEDA_PN" ""
+			(at 250.19 22.86 0)
+			(hide yes)
+			(show_name no)
+			(do_not_autoplace no)
+			(effects
+				(font
+					(size 1.27 1.27)
+				)
+			)
+		)
+		(pin "2"
+		)
+		(pin "1"
+		)
+		(instances
+			(project "digiradio-batch2"
+				(path "/b433c945-2781-4d63-86b0-19b6ee138fd9/031d3380-a811-4887-9d07-65b6d0d08041"
+					(reference "C6")
+					(unit 1)
+				)
+			)
+		)
+	)
+	(symbol
 		(lib_id "Device:R")
 		(at 175.26 100.33 270)
@@
 			)
 		)
-		(property "Value" "25AA1024-I_SM"
+		(property "Value" "25AA1024-I/SM"
 			(at 246.38 113.03 0)
 			(show_name no)
@@
 			)
 		)
-		(property "Footprint" "MIKILAB_25AA1024:SOIC127P600X175-8N"
+		(property "Footprint" "Package_SO:SOIC-8_5.3x5.3mm_P1.27mm"
 			(at 246.38 130.81 0)
 			(hide yes)
@@
 			)
 		)
-		(property "PNM" "25AA1024-I_SM"
+		(property "PNM" "25AA1024-I/SM"
 			(at 246.38 130.81 0)
 			(hide yes)
@@
 			)
 		)
-		(property "Value" "12pF"
+		(property "Value" "15pF"
 			(at 27.178 170.942 90)
 			(show_name no)
@@
 			)
 		)
-		(property "Description" "12pF X7R ±10% 50V 0603 Ceramic Capacitors RoHS"
+		(property "Description" "CAP CER 15pF 50V NP0 0603"
 			(at 24.13 171.45 0)
 			(hide yes)
@@
 			)
 		)
-		(property "PNM" "C0603C120K5RACTU"
+		(property "PNM" "CC0603JRNPO9BN150"
 			(at 24.13 171.45 90)
 			(hide yes)
@@
 			)
 		)
-		(property "Value" "12pF"
+		(property "Value" "15pF"
 			(at 53.848 169.672 90)
 			(show_name no)
@@
 			)
 		)
-		(property "Description" "12pF X7R ±10% 50V 0603 Ceramic Capacitors RoHS"
+		(property "Description" "CAP CER 15pF 50V NP0 0603"
 			(at 50.8 170.18 0)
 			(hide yes)
@@
 			)
 		)
-		(property "PNM" "C0603C120K5RACTU"
+		(property "PNM" "CC0603JRNPO9BN150"
 			(at 50.8 170.18 90)
 			(hide yes)

Commit message: Add the TOSLINK output to the v2 board
Fit an Everlight PLT237/T10WH as J5 on the top edge, driven from
ADAU1452 SPDIFOUT through R56, with FB3 and C65 on its 3V3_AUDIO
supply. The optical face sits 2.31 mm past the board edge.

Move flash U3 and its parts next to U8 and U13 to free the edge, which
shortens the M_SPI traces from 80-95 mm to 34-46 mm.

Pin order follows the LCSC footprint: pad 1 Vin, 2 Vcc, 3 GND.

Co-Authored-By: Claude <noreply@anthropic.com>
Parts:
- added C65: 100nF, Capacitor_SMD:C_0603_1608Metric, symbol Device:C
- added FB3: BLM18SG121TN1D, Inductor_SMD:L_0603_1608Metric, symbol Device:FerriteBead
- added J5: PLT237/T10WH, MIKILAB_FCR684205R:PLT237_T10WH, symbol MIKILAB_FCR684205R:PLT237_T10WH
- added R56: 33, Resistor_SMD:R_0603_1608Metric, symbol Device:R
- C141, C142: value 15pF -> 12pF; PNM CC0603JRNPO9BN150 -> CC0603JRNPO9BN120
Connections:
- net 3V3_AUDIO: now also FB3.1
- net GND: now also C65.1, J5.3 (GND)
- net SPDIFOUT: now reaches U13.5 (SPDIFOUT)
- net SPDIFOUT: now also R56.2
- new net: J5.1 (VIN), R56.1
- new net: C65.2, FB3.2, J5.2 (VCC)
- no-connect marks 22 -> 21
