File: Hardware-v2/kicad/digiradio-batch2.kicad_pcb (KiCad board)
At the start: 6 copper layers, 60 x 80 mm, 172 parts, among them J1 USB_C_Receptacle_USB2.0_16P, J2 SMA-KE-P, J3 BAT, J5 PLT237/T10WH, U1 24AA025E64, U10 BQ25896RTWT, U11 TPS63031DSKR, U12 TPS7A2018PDBVR, U13 ADAU1452, U14 25AA1024-I/SM, U2 ESP32-S31-WROOM-3, U3 W25Q128JVS, U4 TLV62568DBV, U5 TPS63031DSKR, U6 FSC-BT1058, U7 W25Q16JW, U8 Si4684-A10-GM, U9 MAX17048G_T10, Y2 ABM8-19.200MHZ-10-1-U-T, Y3 ABM3B-12.288MHZ-10-1-U-T

Commit message: Set C10 to 1 uF and update the v2 schematic PDF
Michele's schematic edit changes C10 from 100 nF to 1 uF. The PCB now matches
it, and the PDF is exported from the current schematic, including the new J2.

Co-Authored-By: Claude Opus 5.5 (1M context) <noreply@anthropic.com>
Parts:
- C10: value 100nF -> 1uF
Changed lines of the file:
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@@
 			)
 		)
-		(property "Value" "100nF"
+		(property "Value" "1uF"
 			(at 0 1.43 0)
 			(layer "F.Fab")
@@
 			)
 		)
-		(property "Description" "CAP CER 100nF 50V ±10% X7R 0603"
+		(property "Description" "CAP CER 1uF 50V X7R 0603"
 			(at 0 0 0)
 			(layer "F.Fab")
@@
 			)
 		)
-		(property "PNM" "CC0603KRX7R9BB104"
+		(property "PNM" "CL10B105KB8NQNC"
 			(at 0 0 0)
 			(unlocked yes)
