File: Hardware-v2/kicad/power-engine.kicad_sch (KiCad schematic)
At the start: 57 parts, among them J3 BAT, U10 BQ25896RTWT, U11 TPS63031DSKR, U12 TPS7A2018PDBVR, U4 TLV62568DBV, U5 TPS63031DSKR, U9 MAX17048G_T10

Commit message: Set C10 to 1 uF and update the v2 schematic PDF
Michele's schematic edit changes C10 from 100 nF to 1 uF. The PCB now matches
it, and the PDF is exported from the current schematic, including the new J2.

Co-Authored-By: Claude Opus 5.5 (1M context) <noreply@anthropic.com>
Parts:
- C10: value 100nF -> 1uF; PNM CC0603KRX7R9BB104 -> CL10B105KB8NQNC
Changed lines of the file:
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@@
 			)
 		)
-		(property "Value" "100nF"
+		(property "Value" "1uF"
 			(at 224.028 25.146 0)
 			(show_name no)
@@
 			)
 		)
-		(property "Description" "CAP CER 100nF 50V ±10% X7R 0603"
+		(property "Description" "CAP CER 1uF 50V X7R 0603"
 			(at 223.52 22.86 0)
 			(hide yes)
@@
 			)
 		)
-		(property "PNM" "CC0603KRX7R9BB104"
+		(property "PNM" "CL10B105KB8NQNC"
 			(at 223.52 22.86 0)
 			(hide yes)
